File: relayChain5.brd (EAGLE design)
At the start: 123 x 62 mm, 48 parts, among them IC1 TPIC6B595DWRG4, J1 ACJM-HHDR, J10 ACJM-MHDEM, J11 ACJM-HHDR, J2 9V, J3 MOLEX-PICO-LOCK-1X08, J4 ACJM-MHDEM, J5 ACJM-MHDEM, J6 ACJM-MHDEM, J8 MOLEX-PICO-LOCK-1X04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

Commit message: finished initial design
Parts:
- moved R4 26.0 mm to (30.2, 15.4), turned to 180 degrees
- moved J7 18.8 mm to (42.8, 13.7)
- moved C7 14.1 mm to (36.1, 14.9)
- moved R7 5.06 mm to (47.6, 7.80), turned to 90 degrees
- moved OK1 2.21 mm to (115.8, 16.3), turned to 90 degrees
- moved R6 1.49 mm to (44.6, 6.50), turned to 90 degrees
- moved R2 0.34 mm to (94.4, 4.33)
Routing:
- net RELAY_0: track 14.0 -> 99.8 mm
- net SRCK: track 0.00 -> 80.5 mm, vias 0 -> 2
- net RCK: track 0.00 -> 79.5 mm, vias 0 -> 2
- net RELAY_1: track 14.3 -> 84.0 mm
- net DATA: track 0.00 -> 69.3 mm, vias 0 -> 2
- net RELAY_2: track 14.6 -> 68.7 mm
- net CE: track 0.00 -> 50.7 mm
- net CSN: track 0.00 -> 48.4 mm
- net MOSI: track 0.00 -> 42.3 mm
- net MISO: track 0.00 -> 39.9 mm
- net SCK: track 0.00 -> 38.6 mm, vias 0 -> 2
- net RELAY_3: track 14.6 -> 53.1 mm
- net SIG_OUT: track 0.00 -> 34.6 mm
- net 5V: track 80.1 -> 109.7 mm, vias 15 -> 17
- net RELAY_4: track 14.8 -> 33.7 mm
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